File: HARDWARE/ekoenergo.kicad_sch (KiCad schematic)
At the start: 36 parts, among them J1 WSH500, J2 DC+, J3 EARTH, J4 DC-, J5 A, J6 B, Q1 47n60, Q2 47n60, Q3 47n60, Q4 47n60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

Commit message: update
Parts:
- removed J1: WSH500, zvt:WSH500, symbol zvt:WSH500
- added U1: WS3081, fab_U:SOP-8_3.9x4.9mm_P1.27mm, symbol fab_U:WS3081
- added U2: WSH500, zvt:WSH500, symbol zvt:WSH500
- Q1, Q2, Q3, Q4: footprint fab_T:TO-247-3_Horizontal_TabDown_Cut -> Package_TO_SOT_THT:TO-247-3_Vertical
Connections:
- net A1: now also R34.1, R35.2; no longer R29.1
- net A2: now also R29.1; no longer R34.1, R35.2
- net OUT_A: now also U2.37 (T1G), U2.38 (T1G)
- net OUT_B: now also U2.45 (T3G), U2.46 (T3G)
- net T1: now also U2.35 (T1), U2.36 (T1)
- net T2: now also U2.41 (T2), U2.42 (T2)
- net T3: now also U2.43 (T3), U2.44 (T3)
- net T4: now also U2.49 (T4), U2.50 (T4)
- new net: U2.39 (T2G), U2.40 (T2G)
- new net: U2.47 (T4G), U2.48 (T4G)
Other:
- note added: "current measurement"
- note added: "voltage measurement"
- note removed: "meranie napätia"
- note removed: "meranie prúdu"
- moved on the sheet: C12, C18, C19, C20, C21, C22, C23, D12, D17, J2, J3, J4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

Commit message: update
Parts:
- removed Q1, Q2, Q3, Q4: 47n60, Package_TO_SOT_THT:TO-247-3_Vertical, symbol Transistor_FET:C2M0040120D
- removed Rm1: 0,013, Resistor_SMD:R_2816_7142Metric, symbol fabrika_lib:R
- added C1: 100n, Capacitor_SMD:C_0805_2012Metric, symbol fabrika_lib:C
- added C2: 1n, Capacitor_SMD:C_0805_2012Metric, symbol fabrika_lib:C
- added Q1, Q2, Q3, Q4: 47N60, fab_T:TO-247-3_Horizontal_TabDown_Cut, symbol fab_T:47N60
- added R1: 560/1%, Resistor_SMD:R_0805_2012Metric, symbol fabrika_lib:R
- added U3: ACS712ELCTR-20A-T, Package_SO:SOIC-8_3.9x4.9mm_P1.27mm, symbol fabrika_lib:ACS712
- J5: value A -> B
- J6: value B -> A
- U2: footprint zvt:WSH500 -> zvt:WSH500_SMD
Connections:
- net +5V: now also C1.1
- net A1: now also U2.30 (AI1)
- net A2: now also U2.31 (AI2), R1.1
- net DC+: now also Q1.2 (D), Q3.2 (D)
- net DC-: no longer C19.2, C20.2, C21.2, D17.1 (K)
- net GND: now also C19.2, C20.2, C21.2, D17.1 (K), C1.2, C2.2, U3.1 (IP+), U3.2 (IP+)
- net OUT_A: now also Q1.3 (S), Q2.2 (D); no longer U2.37 (T1G), U2.38 (T1G)
- net OUT_B: now also Q3.3 (S), Q4.2 (D); no longer U2.45 (T3G), U2.46 (T3G)
- net T1: now also Q1.1 (G); no longer U2.35 (T1), U2.36 (T1)
- net T2: now also Q2.1 (G); no longer U2.41 (T2), U2.42 (T2)
- net T3: now also Q3.1 (G); no longer U2.43 (T3), U2.44 (T3)
- net T4: now also Q4.1 (G); no longer U2.49 (T4), U2.50 (T4)
- net _mer: now also Q2.3 (S), Q4.3 (S), U3.3 (IP-), U3.4 (IP-)
- new net: U2.35 (T1), U2.36 (T1)
- new net: U2.37 (T1G), U2.38 (T1G)
- new net: U2.41 (T2), U2.42 (T2)
- new net: U2.43 (T3), U2.44 (T3)
- new net: U2.45 (T3G), U2.46 (T3G)
- new net: U2.49 (T4), U2.50 (T4)
Other:
- note removed: "current measurement"
- moved on the sheet: C19, C20, C21, C22, C23, C25, D22, D23, D24, J5, J6, R19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

Commit message: update
Parts:
- removed U1: WS3081, fab_U:SOP-8_3.9x4.9mm_P1.27mm, symbol fab_U:WS3081
Connections:
- net A2 is gone; now on net A1: R1.1, R29.1, U2.31 (AI2)
- net +5V: now also U3.6 (FILTER)
- net A1: now also U2.29 (AI0)
- net OUT_A: now also U2.37 (T1G), U2.38 (T1G)
- net OUT_B: now also U2.45 (T3G), U2.46 (T3G)
- net T1: now also U2.35 (T1), U2.36 (T1)
- net T2: now also U2.41 (T2), U2.42 (T2)
- net T3: now also U2.43 (T3), U2.44 (T3)
- net T4: now also U2.49 (T4), U2.50 (T4)
- net at R1.2: now also U3.7 (VIOUT)
- net at U3.8 (VCC): now also C2.1
Other:
- moved on the sheet: C1, C2, R1, U2

Commit message: update
Parts:
- added U1: TCA9555PWR, Package_SO:TSSOP-24_4.4x7.8mm_P0.65mm, symbol Interface_Expansion:TCA9555PWR
Changed lines of the file:
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@@
+	)
+	(symbol
+		(lib_id "Interface_Expansion:TCA9555PWR")
+		(at 113.03 210.82 0)
+		(unit 1)
+		(exclude_from_sim no)
+		(in_bom yes)
+		(on_board yes)
+		(dnp no)
+		(fields_autoplaced yes)
+		(property "Reference" "U1"
+			(at 115.1733 182.88 0)
+			(effects
+				(font
+					(size 1.27 1.27)
+				)
+				(justify left)
+			)
+		)
+		(property "Value" "TCA9555PWR"
+			(at 115.1733 185.42 0)
+			(effects
+				(font
+					(size 1.27 1.27)
+				)
+				(justify left)
+			)
+		)
+		(property "Footprint" "Package_SO:TSSOP-24_4.4x7.8mm_P0.65mm"
+			(at 139.7 236.22 0)
+			(effects
+				(font
+					(size 1.27 1.27)
+				)
+				(hide yes)
+			)
+		)
+		(property "Datasheet" "http://www.ti.com/lit/ds/symlink/tca9555.pdf"
+			(at 100.33 187.96 0)
+			(effects
+				(font
+					(size 1.27 1.27)
+				)
+				(hide yes)
+			)
+		)
+		(property "Description" "16-bit I/O expander, I2C and SMBus interface, interrupts, w/ pull-ups, TSSOP-24 package"
+			(at 113.03 210.82 0)
+			(effects
+				(font
+					(size 1.27 1.27)
+				)
+				(hide yes)
+			)
+		)
+		(pin "23"
+		)
+		(pin "1"
+		)
+		(pin "10"
+		)
+		(pin "5"
+		)
+		(pin "17"
+		)
+		(pin "8"
+		)
+		(pin "13"
+		)
+		(pin "4"
+		)
+		(pin "9"
+		)
+		(pin "12"
+		)
+		(pin "6"
+		)
+		(pin "19"
+		)
+		(pin "24"
+		)
+		(pin "7"
+		)
+		(pin "22"
+		)
+		(pin "11"
+		)
+		(pin "15"
+		)
+		(pin "3"
+		)
+		(pin "16"
+		)
+		(pin "14"
+		)
+		(pin "2"
+		)
+		(pin "21"
+		)
+		(pin "18"
+		)
+		(pin "20"
+		)
+		(instances
+			(project ""
+				(path "/0cd79e19-f12f-4f42-8abd-ff75db712464"
+					(reference "U1")
+					(unit 1)
+				)
+			)
+		)
 	)
 	(symbol
