File: HARDWARE/ekoenergo.kicad_pcb (KiCad board)
At the start: 4 copper layers, 110 x 80 mm, 33 parts, among them J1 WSH500, J2 DC+, J3 EARTH, J4 DC-, J5 A, J6 B, Q1 47n60, Q2 47n60, Q3 47n60, Q4 47n60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

Commit message: Update ekoenergo.kicad_pcb
Connections:
- J1 pad 39: /T3 -> unconnected-(J1-Pin_39-Pad39)
- J1 pad 41: /OUT_B -> unconnected-(J1-Pin_41-Pad41)
- J1 pad 47: /T4 -> unconnected-(J1-Pin_47-Pad47)
Changed lines of the file:
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@@
 	(net 45 "unconnected-(J1-Pin_32-Pad32)")
 	(net 46 "unconnected-(J1-Pin_38-Pad38)")
+	(net 47 "unconnected-(J1-Pin_47-Pad47)")
+	(net 48 "unconnected-(J1-Pin_39-Pad39)")
+	(net 49 "unconnected-(J1-Pin_41-Pad41)")
 	(footprint "Resistor_SMD:R_0805_2012Metric"
 		(layer "F.Cu")
@@
 		(property ki_fp_filters "R_*")
 		(sheetname "/")
-		(sheetfile "WSH550.kicad_sch")
+		(sheetfile "ekoenergo.kicad_sch")
 		(attr smd)
 		(fp_line
@@
 		(property ki_fp_filters "MountingHole*Pad*")
 		(sheetname "/")
-		(sheetfile "WSH550.kicad_sch")
+		(sheetfile "ekoenergo.kicad_sch")
 		(attr exclude_from_pos_files exclude_from_bom)
 		(fp_circle
@@
 		(property ki_fp_filters "R_*")
 		(sheetname "/")
-		(sheetfile "WSH550.kicad_sch")
+		(sheetfile "ekoenergo.kicad_sch")
 		(attr smd)
 		(fp_line
@@
 		(property ki_fp_filters "TO?247*")
 		(sheetname "/")
-		(sheetfile "WSH550.kicad_sch")
+		(sheetfile "ekoenergo.kicad_sch")
 		(attr through_hole)
 		(fp_line
@@
 		(property ki_fp_filters "D?DO?201AE*")
 		(sheetname "/")
-		(sheetfile "WSH550.kicad_sch")
+		(sheetfile "ekoenergo.kicad_sch")
 		(attr through_hole)
 		(fp_line
@@
 		)
 		(sheetname "/")
-		(sheetfile "WSH550.kicad_sch")
+		(sheetfile "ekoenergo.kicad_sch")
 		(attr smd)
 		(fp_line
@@
 		(property ki_fp_filters "TerminalBlock*:*")
 		(sheetname "/")
-		(sheetfile "WSH550.kicad_sch")
+		(sheetfile "ekoenergo.kicad_sch")
 		(attr through_hole)
 		(fp_rect
@@
 		(property ki_fp_filters "C_*")
 		(sheetname "/")
-		(sheetfile "WSH550.kicad_sch")
+		(sheetfile "ekoenergo.kicad_sch")
 		(attr through_hole)
 		(fp_line
@@
 		(property ki_fp_filters "R_*")
 		(sheetname "/")
-		(sheetfile "WSH550.kicad_sch")
+		(sheetfile "ekoenergo.kicad_sch")
 		(attr smd)
 		(fp_line
@@
 		(property ki_fp_filters "TerminalBlock*:*")
 		(sheetname "/")
-		(sheetfile "WSH550.kicad_sch")
+		(sheetfile "ekoenergo.kicad_sch")
 		(attr through_hole)
 		(fp_rect
@@
 		(property ki_fp_filters "R_*")
 		(sheetname "/")
-		(sheetfile "WSH550.kicad_sch")
+		(sheetfile "ekoenergo.kicad_sch")
 		(attr smd)
 		(fp_line
@@
 		(property ki_fp_filters "TO?247*")
 		(sheetname "/")
-		(sheetfile "WSH550.kicad_sch")
+		(sheetfile "ekoenergo.kicad_sch")
 		(attr through_hole)
 		(fp_line
@@
 		(property ki_fp_filters "TerminalBlock*:*")
 		(sheetname "/")
-		(sheetfile "WSH550.kicad_sch")
+		(sheetfile "ekoenergo.kicad_sch")
 		(attr through_hole)
 		(fp_rect
@@
 		(property ki_fp_filters "C_*")
 		(sheetname "/")
-		(sheetfile "WSH550.kicad_sch")
+		(sheetfile "ekoenergo.kicad_sch")
 		(attr through_hole)
 		(fp_line
@@
 		(property ki_fp_filters "C_*")
 		(sheetname "/")
-		(sheetfile "WSH550.kicad_sch")
+		(sheetfile "ekoenergo.kicad_sch")
 		(attr smd)
 		(fp_line
@@
 		(property ki_fp_filters "LED* LED_SMD:* LED_THT:*")
 		(sheetname "/")
-		(sheetfile "WSH550.kicad_sch")
+		(sheetfile "ekoenergo.kicad_sch")
 		(attr smd)
 		(fp_line
@@
 		(property ki_fp_filters "LED* LED_SMD:* LED_THT:*")
 		(sheetname "/")
-		(sheetfile "WSH550.kicad_sch")
+		(sheetfile "ekoenergo.kicad_sch")
 		(attr smd)
 		(fp_line
@@
 		(property ki_fp_filters "C_*")
 		(sheetname "/")
-		(sheetfile "WSH550.kicad_sch")
+		(sheetfile "ekoenergo.kicad_sch")
 		(attr through_hole)
 		(fp_line
@@
 		(property ki_fp_filters "C_*")
 		(sheetname "/")
-		(sheetfile "WSH550.kicad_sch")
+		(sheetfile "ekoenergo.kicad_sch")
 		(attr smd)
 		(fp_line
@@
 		(property ki_fp_filters "MountingHole*Pad*")
 		(sheetname "/")
-		(sheetfile "WSH550.kicad_sch")
+		(sheetfile "ekoenergo.kicad_sch")
 		(attr exclude_from_pos_files exclude_from_bom)
 		(fp_circle
@@
 		)
 		(sheetname "/")
-		(sheetfile "WSH550.kicad_sch")
+		(sheetfile "ekoenergo.kicad_sch")
 		(attr smd)
 		(fp_line
@@
 		(property ki_fp_filters "R_*")
 		(sheetname "/")
-		(sheetfile "WSH550.kicad_sch")
+		(sheetfile "ekoenergo.kicad_sch")
 		(attr smd)
 		(fp_line
@@
 		(property ki_fp_filters "TerminalBlock*:*")
 		(sheetname "/")
-		(sheetfile "WSH550.kicad_sch")
+		(sheetfile "ekoenergo.kicad_sch")
 		(attr through_hole)
 		(fp_rect
@@
 		(property ki_fp_filters "MountingHole*Pad*")
 		(sheetname "/")
-		(sheetfile "WSH550.kicad_sch")
+		(sheetfile "ekoenergo.kicad_sch")
 		(attr exclude_from_pos_files exclude_from_bom)
 		(fp_circle
@@
 		(property ki_fp_filters "C_*")
 		(sheetname "/")
-		(sheetfile "WSH550.kicad_sch")
+		(sheetfile "ekoenergo.kicad_sch")
 		(attr through_hole)
 		(fp_line
@@
 		(property ki_fp_filters "MountingHole*Pad*")
 		(sheetname "/")
-		(sheetfile "WSH550.kicad_sch")
+		(sheetfile "ekoenergo.kicad_sch")
 		(attr exclude_from_pos_files exclude_from_bom)
 		(fp_circle
@@
 		(property ki_fp_filters "LED* LED_SMD:* LED_THT:*")
 		(sheetname "/")
-		(sheetfile "WSH550.kicad_sch")
+		(sheetfile "ekoenergo.kicad_sch")
 		(attr smd)
 		(fp_line
@@
 		(property ki_fp_filters "TerminalBlock*:*")
 		(sheetname "/")
-		(sheetfile "WSH550.kicad_sch")
+		(sheetfile "ekoenergo.kicad_sch")
 		(attr through_hole)
 		(fp_rect
@@
 		(property ki_fp_filters "TO?247*")
 		(sheetname "/")
-		(sheetfile "WSH550.kicad_sch")
+		(sheetfile "ekoenergo.kicad_sch")
 		(attr through_hole)
 		(fp_line
@@
 		(property ki_fp_filters "TO?247*")
 		(sheetname "/")
-		(sheetfile "WSH550.kicad_sch")
+		(sheetfile "ekoenergo.kicad_sch")
 		(attr through_hole)
 		(fp_line
@@
 		)
 		(sheetname "/")
-		(sheetfile "WSH550.kicad_sch")
+		(sheetfile "ekoenergo.kicad_sch")
 		(attr through_hole)
 		(fp_line
@@
 			(layers "*.Cu" "*.Mask")
 			(remove_unused_layers no)
-			(net 5 "/T3")
-			(pinfunction "T3")
+			(net 48 "unconnected-(J1-Pin_39-Pad39)")
+			(pinfunction "Pin_39")
 			(pintype "passive")
 		)
@@
 			(layers "*.Cu" "*.Mask")
 			(remove_unused_layers no)
-			(net 3 "/OUT_B")
-			(pinfunction "T3G")
-			(pintype "output")
+			(net 49 "unconnected-(J1-Pin_41-Pad41)")
+			(pinfunction "Pin_41")
+			(pintype "passive")
 		)
 		(pad "42" thru_hole circle
@@
 			(layers "*.Cu" "*.Mask")
 			(remove_unused_layers no)
-			(net 6 "/T4")
-			(pinfunction "T4")
-			(pintype "output")
+			(net 47 "unconnected-(J1-Pin_47-Pad47)")
+			(pinfunction "Pin_47")
+			(pintype "passive")
 		)
 		(pad "48" thru_hole circle
@@
 		(property ki_fp_filters "C_*")
 		(sheetname "/")
-		(sheetfile "WSH550.kicad_sch")
+		(sheetfile "ekoenergo.kicad_sch")
 		(attr through_hole)
 		(fp_line
@@
 		(property ki_fp_filters "R_*")
 		(sheetname "/")
-		(sheetfile "WSH550.kicad_sch")
+		(sheetfile "ekoenergo.kicad_sch")
 		(attr smd)
 		(fp_line
