File: HARDWARE/ekoenergo.kicad_pcb (KiCad board)
At the start: 4 copper layers, 110 x 80 mm, 33 parts, among them J1 WSH500, J2 DC+, J3 EARTH, J4 DC-, J5 A, J6 B, Q1 47n60, Q2 47n60, Q3 47n60, Q4 47n60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

Commit message: update
Routing:
- net /T3: track 0.00 -> 6.40 mm
Changed lines of the file:
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@@
+	)
+	(segment
+		(start 140.045 102.645)
+		(end 140.88 101.81)
+		(width 0.2)
+		(layer "F.Cu")
+		(net 5)
+	)
+	(segment
+		(start 140.045 107.867)
+		(end 140.045 102.645)
+		(width 0.2)
+		(layer "F.Cu")
+		(net 5)
 	)
 	(segment

Commit message: update
Parts:
- removed J1: WSH500, zvt:WSH500
- removed Rm1: 0,013, Resistor_SMD:R_2816_7142Metric
- added C1: 100n, Capacitor_SMD:C_0805_2012Metric, F.Cu at (84.8, 115.1)
- added C2: 1n, Capacitor_SMD:C_0805_2012Metric, F.Cu at (84.8, 118.1)
- added R1: 560/1%, Resistor_SMD:R_0805_2012Metric, F.Cu at (89.3, 115.0)
- added U1: WS3081, fab_U:SOP-8_3.9x4.9mm_P1.27mm, F.Cu at (236.3, 74.4)
- added U2: WSH500, zvt:WSH500_SMD, F.Cu at (177.6, 108.1)
- added U3: ACS712ELCTR-20A-T, Package_SO:SOIC-8_3.9x4.9mm_P1.27mm, F.Cu at (132.1, 93.5)
- J3: renamed from J6; value B -> EARTH
- J5: value A -> B
- J6: renamed from J3; value EARTH -> A
- Q1: renamed from Q2; value 47n60 -> 47N60
- Q2: renamed from Q1; value 47n60 -> 47N60
- Q3: renamed from Q4; value 47n60 -> 47N60
- Q4: renamed from Q3; value 47n60 -> 47N60
- moved C18 102.7 mm to (222.3, 123.9), turned to 0 degrees
- moved C12 37.6 mm to (84.9, 101.6)
- moved J3 28.0 mm to (177.9, 132.8)
- moved Q1 26.0 mm to (168.9, 101.8)
- moved Q2 26.0 mm to (150.9, 101.8)
- moved Q3 26.0 mm to (132.9, 101.8)
- moved Q4 26.0 mm to (114.9, 101.8)
- moved J5 22.0 mm to (114.9, 132.8)
- moved J6 13.0 mm to (149.9, 132.8)
- moved J2 10.0 mm to (165.9, 132.8)
- moved U5 6.36 mm to (196.9, 122.7)
- moved J4 1.00 mm to (189.9, 132.8)
Connections:
- C19 pad 2: /DC- -> GND
- C20 pad 2: /DC- -> GND
- C21 pad 2: /DC- -> GND
- D17 pad 1: /DC- -> GND
- J3 pad 1: /OUT_A -> Earth
- J6 pad 1: Earth -> /OUT_A
- Q1 pad 1: /T2 -> /T1
- Q1 pad 2: /OUT_A -> /DC+
- Q1 pad 3: /_mer -> /OUT_A
- Q2 pad 1: /T1 -> /T2
- Q2 pad 2: /DC+ -> /OUT_A
- Q2 pad 3: /OUT_A -> /_mer
- Q3 pad 1: /T4 -> /T3
- Q3 pad 2: /OUT_B -> /DC+
- Q3 pad 3: /_mer -> /OUT_B
- Q4 pad 1: /T3 -> /T4
- Q4 pad 2: /DC+ -> /OUT_B
- Q4 pad 3: /OUT_B -> /_mer
- R29 pad 1: /A1 -> /A2
- R34 pad 1: /A2 -> /A1
- R35 pad 2: /A2 -> /A1
Routing:
- net /T3: track 6.40 -> 0.00 mm
- net /T1: track 1.23 -> 0.00 mm
- added copper zone on B.Cu, net /DC+
- added copper zone on F.Cu, net /DC-
- added copper zone on F.Cu, net /_mer
- added copper zone on F.Cu, net GND
- removed copper zone on F.Cu, net /DC+
- removed copper zone on B.Cu, net /DC-
- removed copper zone on B.Cu, net /_mer

Commit message: update
Parts:
- moved C12 152.8 mm to (236.6, 118.9), turned to 180 degrees
- moved U1 93.4 mm to (154.8, 120.1)
- moved U2 10.5 mm to (188.1, 108.1)
- moved C18 8.11 mm to (225.0, 131.6)
Connections:
- C2 pad 1: unconnected-(C2-Pad1) -> Net-(U3-VCC)
- R1 pad 1: /A2 -> /A1
- R1 pad 2: unconnected-(R1-Pad2) -> Net-(U3-VIOUT)
- R29 pad 1: /A2 -> /A1
- U2 pad 29: unconnected-(U2-AI0-Pad29) -> /A1
- U2 pad 31: /A2 -> /A1
- U2 pad 35: Net-(U2-T1-Pad35) -> /T1
- U2 pad 36: Net-(U2-T1-Pad35) -> /T1
- U2 pad 37: Net-(U2-T1G-Pad37) -> /OUT_A
- U2 pad 38: Net-(U2-T1G-Pad37) -> /OUT_A
- U2 pad 41: Net-(U2-T2-Pad41) -> /T2
- U2 pad 42: Net-(U2-T2-Pad41) -> /T2
- U2 pad 43: Net-(U2-T3-Pad43) -> /T3
- U2 pad 44: Net-(U2-T3-Pad43) -> /T3
- U2 pad 45: Net-(U2-T3G-Pad45) -> /OUT_B
- U2 pad 46: Net-(U2-T3G-Pad45) -> /OUT_B
- U2 pad 49: Net-(U2-T4-Pad49) -> /T4
- U2 pad 50: Net-(U2-T4-Pad49) -> /T4
- U3 pad 6: unconnected-(U3-FILTER-Pad6) -> +5V
- U3 pad 7: unconnected-(U3-VIOUT-Pad7) -> Net-(U3-VIOUT)
- U3 pad 8: unconnected-(U3-VCC-Pad8) -> Net-(U3-VCC)
Routing:
- net /T1: track 0.00 -> 42.1 mm
- net /T2: track 0.00 -> 31.7 mm
- net /OUT_B: track 0.00 -> 16.5 mm
- net /T3: track 0.00 -> 16.3 mm
- net /T4: track 0.00 -> 12.0 mm
Other:
- board size 110 x 80 mm -> 120 x 80 mm
